Commit message: ..,

File: phantom_description/urdf/phantomX_model.xacro (robot description, xacro)
@@ -127,5 +127,5 @@
 			<parent link="coxa_${side}${position}" />
 			<child link="femur_${side}${position}" />
-			<axis xyz="0.0 0.0 ${-axis}" />
+			<axis xyz="0.0 0.0 ${axis}" />
 			<limit lower="${joint_lower_limit}" upper="${joint_upper_limit}" effort="${joint_effort}" velocity="${joint_velocity}" />
 		</joint>
@@ -176,5 +176,5 @@
 			<parent link="femur_${side}${position}" />
 			<child link="tibia_${side}${position}" />
-			<axis xyz="0.0 0.0 ${axis}" />
+			<axis xyz="0.0 0.0 ${-axis}" />
 			<limit lower="${joint_lower_limit}" upper="${joint_upper_limit}" effort="${joint_effort}" velocity="${joint_velocity}" />
 		</joint>

Commit message: add model.urdf

File: phantom_description/urdf/phantomX_model.xacro (robot description, xacro)
@@ -50,4 +50,101 @@
         <material>Gazebo/DarkGrey</material>
     </gazebo>
+	<!-- Head Pan and Tilt properties -->
+	<joint name="head_pan_joint" type="revolute">
+		<parent link="body_link"/>
+		<child link="head_pan_link"/>
+		<axis xyz="0.0 0.0 1.0" />
+		<origin xyz="0.145 0.0 0.080" />
+		<limit lower="-${3.14}" upper="${3.14}" effort="10000" velocity="100" />
+	</joint>
+	<link name="head_pan_link">
+        <inertial>
+            <origin xyz="0.0 0.0 0.0" rpy="0.0 0.0 0.0" />
+            <mass value="0.00001"/>
+            <inertia
+                ixx="1.0" ixy="0.0"  ixz="0.0"
+                iyy="1.0" iyz="0.0"
+                izz="1.0" />
+        </inertial>
+    </link>
+	<joint name="head_tilt_joint" type="revolute">
+		<parent link="head_pan_link"/>
+		<child link="head_tilt_link"/>
+		<axis xyz="0.0 1.0 0.0" />
+		<origin xyz="0.0 0.0 0.020" />
+		<limit lower="-${3.14}" upper="${3.14}" effort="10000" velocity="100" />
+	</joint>
+	<link name="head_tilt_link">
+        <inertial>
+            <origin xyz="0.0 0.0 0.0" rpy="0.0 0.0 0.0" />
+            <mass value="0.00001"/>
+            <inertia
+                ixx="1.0" ixy="0.0"  ixz="0.0"
+                iyy="1.0" iyz="0.0"
+                izz="1.0" />
+        </inertial>
+    </link>
+	<!-- Camera properties -->
+	<joint name="camera_rgb_joint" type="fixed">
+		<parent link="head_tilt_link" />
+		<child link="camera_rgb_optical_frame" />
+		<origin xyz="0.0 0.0 0.0" rpy="${pi/2} ${pi} ${pi/2}" />
+	</joint>
+	<link name="camera_rgb_optical_frame">
+        <inertial>
+            <origin xyz="0.0 0.0 0.0" rpy="0.0 0.0 0.0" />
+            <mass value="0.00001"/>
+            <inertia
+                ixx="1.0" ixy="0.0"  ixz="0.0"
+                iyy="1.0" iyz="0.0"
+                izz="1.0" />
+        </inertial>
+    </link>
+	<joint name="camera_depth_joint" type="fixed">
+		<parent link="head_tilt_link" />
+		<child link="camera_depth_optical_frame" />
+		<origin xyz="0.0 0.0 0.0" rpy="${pi/2} ${pi} ${pi/2}" />
+	</joint>
+	<link name="camera_depth_optical_frame" >
+        <inertial>
+            <origin xyz="0.0 0.0 0.0" rpy="0.0 0.0 0.0" />
+            <mass value="0.00001"/>
+            <inertia
+                ixx="1.0" ixy="0.0"  ixz="0.0"
+                iyy="1.0" iyz="0.0"
+                izz="1.0" />
+        </inertial>
+    </link>
+<joint name="camera_depth_frame" type="fixed">
+	<parent link="head_tilt_link" />
+	<child link="camera_depth_frame_link" />
+	<origin xyz="0.0 0.0 0.0" />
+</joint>
+<link name="camera_depth_frame_link" >
+        <inertial>
+            <origin xyz="0.0 0.0 0.0" rpy="0.0 0.0 0.0" />
+            <mass value="0.00001"/>
+            <inertia
+                ixx="1.0" ixy="0.0"  ixz="0.0"
+                iyy="1.0" iyz="0.0"
+                izz="1.0" />
+        </inertial>
+    </link>
+	<!-- IMU properties -->
+	<joint name="imu_joint" type="fixed">
+		<parent link="base_link" />
+		<child link="imu_link" />
+		<origin xyz="0.0 0.0 0.0" rpy="0.0 0.0 0.0" />
+	</joint>
+	<link name="imu_link">
+        <inertial>
+            <origin xyz="0.0 0.0 0.0" rpy="0.0 0.0 0.0" />
+            <mass value="0.00001"/>
+            <inertia
+                ixx="1.0" ixy="0.0"  ixz="0.0"
+                iyy="1.0" iyz="0.0"
+                izz="1.0" />
+        </inertial>
+    </link>
 	<!-- Joint properties -->
 	<xacro:property name="joint_lower_limit" value="-${3.14}" />
@@ -127,5 +224,5 @@
 			<parent link="coxa_${side}${position}" />
 			<child link="femur_${side}${position}" />
-			<axis xyz="0.0 0.0 ${axis}" />
+			<axis xyz="0.0 0.0 ${-axis}" />
 			<limit lower="${joint_lower_limit}" upper="${joint_upper_limit}" effort="${joint_effort}" velocity="${joint_velocity}" />
 		</joint>
@@ -176,5 +273,5 @@
 			<parent link="femur_${side}${position}" />
 			<child link="tibia_${side}${position}" />
-			<axis xyz="0.0 0.0 ${-axis}" />
+			<axis xyz="0.0 0.0 ${axis}" />
 			<limit lower="${joint_lower_limit}" upper="${joint_upper_limit}" effort="${joint_effort}" velocity="${joint_velocity}" />
 		</joint>

Commit message: hector_slam launch files

File: phantom_description/urdf/phantomX_model.xacro (robot description, xacro)
@@ -50,101 +50,4 @@
         <material>Gazebo/DarkGrey</material>
     </gazebo>
-	<!-- Head Pan and Tilt properties -->
-	<joint name="head_pan_joint" type="revolute">
-		<parent link="body_link"/>
-		<child link="head_pan_link"/>
-		<axis xyz="0.0 0.0 1.0" />
-		<origin xyz="0.145 0.0 0.080" />
-		<limit lower="-${3.14}" upper="${3.14}" effort="10000" velocity="100" />
-	</joint>
-	<link name="head_pan_link">
-        <inertial>
-            <origin xyz="0.0 0.0 0.0" rpy="0.0 0.0 0.0" />
-            <mass value="0.00001"/>
-            <inertia
-                ixx="1.0" ixy="0.0"  ixz="0.0"
-                iyy="1.0" iyz="0.0"
-                izz="1.0" />
-        </inertial>
-    </link>
-	<joint name="head_tilt_joint" type="revolute">
-		<parent link="head_pan_link"/>
-		<child link="head_tilt_link"/>
-		<axis xyz="0.0 1.0 0.0" />
-		<origin xyz="0.0 0.0 0.020" />
-		<limit lower="-${3.14}" upper="${3.14}" effort="10000" velocity="100" />
-	</joint>
-	<link name="head_tilt_link">
-        <inertial>
-            <origin xyz="0.0 0.0 0.0" rpy="0.0 0.0 0.0" />
-            <mass value="0.00001"/>
-            <inertia
-                ixx="1.0" ixy="0.0"  ixz="0.0"
-                iyy="1.0" iyz="0.0"
-                izz="1.0" />
-        </inertial>
-    </link>
-	<!-- Camera properties -->
-	<joint name="camera_rgb_joint" type="fixed">
-		<parent link="head_tilt_link" />
-		<child link="camera_rgb_optical_frame" />
-		<origin xyz="0.0 0.0 0.0" rpy="${pi/2} ${pi} ${pi/2}" />
-	</joint>
-	<link name="camera_rgb_optical_frame">
-        <inertial>
-            <origin xyz="0.0 0.0 0.0" rpy="0.0 0.0 0.0" />
-            <mass value="0.00001"/>
-            <inertia
-                ixx="1.0" ixy="0.0"  ixz="0.0"
-                iyy="1.0" iyz="0.0"
-                izz="1.0" />
-        </inertial>
-    </link>
-	<joint name="camera_depth_joint" type="fixed">
-		<parent link="head_tilt_link" />
-		<child link="camera_depth_optical_frame" />
-		<origin xyz="0.0 0.0 0.0" rpy="${pi/2} ${pi} ${pi/2}" />
-	</joint>
-	<link name="camera_depth_optical_frame" >
-        <inertial>
-            <origin xyz="0.0 0.0 0.0" rpy="0.0 0.0 0.0" />
-            <mass value="0.00001"/>
-            <inertia
-                ixx="1.0" ixy="0.0"  ixz="0.0"
-                iyy="1.0" iyz="0.0"
-                izz="1.0" />
-        </inertial>
-    </link>
-<joint name="camera_depth_frame" type="fixed">
-	<parent link="head_tilt_link" />
-	<child link="camera_depth_frame_link" />
-	<origin xyz="0.0 0.0 0.0" />
-</joint>
-<link name="camera_depth_frame_link" >
-        <inertial>
-            <origin xyz="0.0 0.0 0.0" rpy="0.0 0.0 0.0" />
-            <mass value="0.00001"/>
-            <inertia
-                ixx="1.0" ixy="0.0"  ixz="0.0"
-                iyy="1.0" iyz="0.0"
-                izz="1.0" />
-        </inertial>
-    </link>
-	<!-- IMU properties -->
-	<joint name="imu_joint" type="fixed">
-		<parent link="base_link" />
-		<child link="imu_link" />
-		<origin xyz="0.0 0.0 0.0" rpy="0.0 0.0 0.0" />
-	</joint>
-	<link name="imu_link">
-        <inertial>
-            <origin xyz="0.0 0.0 0.0" rpy="0.0 0.0 0.0" />
-            <mass value="0.00001"/>
-            <inertia
-                ixx="1.0" ixy="0.0"  ixz="0.0"
-                iyy="1.0" iyz="0.0"
-                izz="1.0" />
-        </inertial>
-    </link>
 	<!-- Joint properties -->
 	<xacro:property name="joint_lower_limit" value="-${3.14}" />
