Commit message: Update phantomX_model.xacro

File: phantom_description/urdf/phantomX_model.xacro (robot description, xacro)
@@ -1,93 +1,87 @@
 <?xml version="1.0" encoding="UTF-8" ?>
 <robot xmlns:xacro="http://ros.org/wiki/xacro" name="PhantomX">
-	<!-- parameters -->
-	<xacro:property name="pi" value="3.1415926535897931" />
-	<xacro:property name="body_length_x" value="0.250" />
-	<xacro:property name="body_length_y" value="0.125" />
-	<xacro:property name="coxa_length" value="0.052" />
-	<xacro:property name="femur_length" value="0.065" />
-	<xacro:property name="tibia_length" value="0.133" />
-    <gazebo>
-        <plugin name="gazebo_ros_control" filename="libgazebo_ros_control.so">
-            <robotNamespace>/PhantomX</robotNamespace>
+<!-- parameters -->
+<xacro:property name="pi" value="3.1415926535897931" />
+<xacro:property name="body_length_x" value="0.250" />
+<xacro:property name="body_length_y" value="0.125" />
+<xacro:property name="coxa_length" value="0.052" />
+<xacro:property name="femur_length" value="0.065" />
+<xacro:property name="tibia_length" value="0.133" />
+<gazebo>
+	<plugin name="gazebo_ros_control" filename="libgazebo_ros_control.so">
+        	<robotNamespace>/PhantomX</robotNamespace>
         </plugin>
-    </gazebo>
-    <link name="base_link"/>
-    <joint name="base_joint" type="fixed">
-        <parent link="base_link" />
+</gazebo>
+<link name="base_link"/>
+<joint name="base_joint" type="fixed">
+	<parent link="base_link" />
         <child link="body_link" />
         <origin xyz="0.0 0.0 0.0" rpy="0.0 0.0 0.0" />
-    </joint>
-	<link name="body_link">
-			<visual>
-	  			<origin	xyz="0.0 0.0 0.0" rpy="0.0 0.0 0.0" />
-      			<geometry>
-        			<mesh filename="package://phantom_description/meshes/phantomX/body.stl" scale="0.001 0.001 0.001"/>
-      			</geometry>
-				<material name="">
-					<color rgba="0.7 0.7 0.7 1" />
-				</material>
-			</visual>
-			<collision>
-            <origin xyz="0.0 0.0 0.0" rpy="0.0 0.0 0.0"/>
-            <geometry>
-                <mesh filename="package://phantom_description/meshes/phantomX/body.stl" scale="0.001 0.001 0.001"/>
-            </geometry>
-            <material name="">
-                <color rgba="0.7 0.7 0.7 1"/>
-            </material>
+</joint>
+<link name="body_link">
+	<visual>
+		<origin	xyz="0.0 0.0 0.0" rpy="0.0 0.0 0.0" />
+      		<geometry>
+        		<mesh filename="package://phantom_description/meshes/phantomX/body.stl" scale="0.001 0.001 0.001"/>
+      		</geometry>
+		<material name="">
+			<color rgba="0.7 0.7 0.7 1" />
+		</material>
+	</visual>
+	<collision>
+        	<origin xyz="0.0 0.0 0.0" rpy="0.0 0.0 0.0"/>
+            	<geometry>
+                	<mesh filename="package://phantom_description/meshes/phantomX/body.stl" scale="0.001 0.001 0.001"/>
+            	</geometry>
+            	<material name="">
+                	<color rgba="0.7 0.7 0.7 1"/>
+            	</material>
         </collision>
         <inertial>
             <origin xyz="0.0 0.0 0.0" rpy="0.0 0.0 0.0" />
             <mass value="0.00001"/>
-            <inertia
-                ixx="1.0" ixy="0.0"  ixz="0.0"
-                iyy="1.0" iyz="0.0"
-                izz="1.0" />
+            <inertia ixx="1.0" ixy="0.0"  ixz="0.0" iyy="1.0" iyz="0.0" izz="1.0" />
         </inertial>
-    </link>
-    <gazebo reference="body_link">
-        <material>Gazebo/DarkGrey</material>
-    </gazebo>
-	<!-- Joint properties -->
-	<xacro:property name="joint_lower_limit" value="-${3.14}" />
-	<xacro:property name="joint_upper_limit" value="${3.14}" />
-	<xacro:property name="joint_effort" value="6.0" />
-	<xacro:property name="joint_velocity" value="0.524" />
-	<!-- Leg macro -->
-	<xacro:macro name="leg" params="side position x y angle axis">
-		<!-- leg position -->
-		<joint name="leg_center_joint_${side}${position}" type="fixed">
-			<origin xyz="${x} ${y} 0.0" rpy="0.0 0.0 0.0" />
-			<parent link="body_link" />
-			<child link="leg_center_${side}${position}" />
-		</joint>
-		<link name="leg_center_${side}${position}" >
-            <inertial>
-                <origin xyz="0.0 0.0 0.0" rpy="0.0 0.0 0.0" />
-                <mass value="0.00001"/>
-                <inertia
-                    ixx="1.0" ixy="0.0"  ixz="0.0"
-                    iyy="1.0" iyz="0.0"
-                    izz="1.0" />
-            </inertial>
-        </link>
-		<!-- coxa -->
-		<joint name="coxa_joint_${side}${position}" type="revolute">
-			<origin xyz="0.0 0.0 0.0" rpy="0.0 0.0 ${angle}" />
-			<parent link="leg_center_${side}${position}" />
-			<child link="coxa_${side}${position}" />
-			<axis xyz="0.0 0.0 1.0" />
-			<limit lower="${joint_lower_limit}" upper="${joint_upper_limit}" effort="${joint_effort}" velocity="${joint_velocity}" />
-		</joint>
-		<transmission name="coxa_transmission_${side}${position}">
-            <type>transmission_interface/SimpleTransmission</type>
-            <joint name="coxa_joint_${side}${position}">
-                <hardwareInterface>EffortJointInterface</hardwareInterface>
-            </joint>
-            <actuator name="coxa_motor_${side}${position}">
-                <hardwareInterface>EffortJointInterface</hardwareInterface>
-                <mechanicalReduction>1</mechanicalReduction>
-            </actuator>
+</link>
+<gazebo reference="body_link">
+	<material>Gazebo/DarkGrey</material>
+</gazebo>
+<!-- Joint properties -->
+<xacro:property name="joint_lower_limit" value="-${3.14}" />
+<xacro:property name="joint_upper_limit" value="${3.14}" />
+<xacro:property name="joint_effort" value="6.0" />
+<xacro:property name="joint_velocity" value="0.524" />
+<!-- Leg macro -->
+<xacro:macro name="leg" params="side position x y angle axis">
+	<!-- leg position -->
+	<joint name="leg_center_joint_${side}${position}" type="fixed">
+		<origin xyz="${x} ${y} 0.0" rpy="0.0 0.0 0.0" />
+		<parent link="body_link" />
+		<child link="leg_center_${side}${position}" />
+	</joint>
+	<link name="leg_center_${side}${position}" >
+	        <inertial>
+        	        <origin xyz="0.0 0.0 0.0" rpy="0.0 0.0 0.0" />
+                	<mass value="0.00001"/>
+                	<inertia ixx="1.0" ixy="0.0"  ixz="0.0" iyy="1.0" iyz="0.0" izz="1.0" />
+            	</inertial>
+        </link>
+	<!-- coxa -->
+	<joint name="coxa_joint_${side}${position}" type="revolute">
+		<origin xyz="0.0 0.0 0.0" rpy="0.0 0.0 ${angle}" />
+		<parent link="leg_center_${side}${position}" />
+		<child link="coxa_${side}${position}" />
+		<axis xyz="0.0 0.0 1.0" />
+		<limit lower="${joint_lower_limit}" upper="${joint_upper_limit}" effort="${joint_effort}" velocity="${joint_velocity}" />
+	</joint>
+	<transmission name="coxa_transmission_${side}${position}">
+        	<type>transmission_interface/SimpleTransmission</type>
+        	<joint name="coxa_joint_${side}${position}">
+        		<hardwareInterface>EffortJointInterface</hardwareInterface>
+        	</joint>
+        	<actuator name="coxa_motor_${side}${position}">
+        		<hardwareInterface>EffortJointInterface</hardwareInterface>
+        		<mechanicalReduction>1</mechanicalReduction>
+        	</actuator>
         </transmission>
         <link name="coxa_${side}${position}">
@@ -122,109 +116,103 @@
             <material>Gazebo/DarkGrey</material>
         </gazebo>
-		<!-- femur -->
-		<joint name="femur_joint_${side}${position}" type="revolute">
-			<origin xyz="${coxa_length} 0.0 0.0" rpy="-${pi/2} ${pi/2} 0.0" />
-			<parent link="coxa_${side}${position}" />
-			<child link="femur_${side}${position}" />
-			<axis xyz="0.0 0.0 ${-axis}" />
-			<limit lower="${joint_lower_limit}" upper="${joint_upper_limit}" effort="${joint_effort}" velocity="${joint_velocity}" />
-		</joint>
-		<transmission name="femur_transmission_${side}${position}">
-            <type>transmission_interface/SimpleTransmission</type>
-            <joint name="femur_joint_${side}${position}">
-                <hardwareInterface>EffortJointInterface</hardwareInterface>
-            </joint>
-            <actuator name="femur_motor_${side}${position}">
-                <hardwareInterface>EffortJointInterface</hardwareInterface>
-                <mechanicalReduction>1</mechanicalReduction>
-            </actuator>
+	<!-- femur -->
+	<joint name="femur_joint_${side}${position}" type="revolute">
+		<origin xyz="${coxa_length} 0.0 0.0" rpy="-${pi/2} ${pi/2} 0.0" />
+		<parent link="coxa_${side}${position}" />
+		<child link="femur_${side}${position}" />
+		<axis xyz="0.0 0.0 ${-axis}" />
+		<limit lower="${joint_lower_limit}" upper="${joint_upper_limit}" effort="${joint_effort}" velocity="${joint_velocity}" />
+	</joint>
+	<transmission name="femur_transmission_${side}${position}">
+	        <type>transmission_interface/SimpleTransmission</type>
+        	<joint name="femur_joint_${side}${position}">
+                	<hardwareInterface>EffortJointInterface</hardwareInterface>
+            	</joint>
+            	<actuator name="femur_motor_${side}${position}">
+                	<hardwareInterface>EffortJointInterface</hardwareInterface>
+                	<mechanicalReduction>1</mechanicalReduction>
+            	</actuator>
         </transmission>
         <link name="femur_${side}${position}">
-            <visual>
-                <origin xyz="0.0 0.0 0.0" rpy="0.0 0.0 0.0"/>
-                <geometry>
-                    <mesh filename="package://phantom_description/meshes/phantomX/femur.stl" scale="0.001 0.001 0.001"/>
-                </geometry>
-                <material name="">
-                    <color rgba="0.7 0.7 0.7 1"/>
-                </material>
-            </visual>
-            <collision>
-                <origin xyz="0.0 0.0 0.0" rpy="0.0 0.0 0.0" />
-                <geometry>
-                    <mesh filename="package://phantom_description/meshes/phantomX/femur.stl" scale="0.001 0.001 0.001"/>
-                </geometry>
-                <material name="">
-                    <color rgba="0.7 0.7 0.7 1" />
-                </material>
-            </collision>
-            <inertial>
-                <origin xyz="0.0 0.0 0.0" rpy="0.0 0.0 0.0" />
-                <mass value="0.00001"/>
-                <inertia
-                    ixx="1.0" ixy="0.0"  ixz="0.0"
-                    iyy="1.0" iyz="0.0"
-                    izz="1.0" />
-            </inertial>
+        	<visual>
+                	<origin xyz="0.0 0.0 0.0" rpy="0.0 0.0 0.0"/>
+                	<geometry>
+                    		<mesh filename="package://phantom_description/meshes/phantomX/femur.stl" scale="0.001 0.001 0.001"/>
+                	</geometry>
+                	<material name="">
+                    		<color rgba="0.7 0.7 0.7 1"/>
+                	</material>
+            	</visual>
+            	<collision>
+                	<origin xyz="0.0 0.0 0.0" rpy="0.0 0.0 0.0" />
+                	<geometry>
+                    		<mesh filename="package://phantom_description/meshes/phantomX/femur.stl" scale="0.001 0.001 0.001"/>
+                	</geometry>
+                	<material name="">
+                    		<color rgba="0.7 0.7 0.7 1" />
+                	</material>
+            	</collision>
+            	<inertial>
+                	<origin xyz="0.0 0.0 0.0" rpy="0.0 0.0 0.0" />
+                	<mass value="0.00001"/>
+                	<inertia ixx="1.0" ixy="0.0"  ixz="0.0" iyy="1.0" iyz="0.0" izz="1.0" />
+            	</inertial>
         </link>
         <gazebo reference="femur_${side}${position}">
-            <material>Gazebo/DarkGrey</material>
+        	<material>Gazebo/DarkGrey</material>
         </gazebo>
-		<!-- tibia -->
-		<joint name="tibia_joint_${side}${position}" type="revolute">
-			<origin xyz="0.0 -${femur_length} 0.0" rpy="${pi} 0.0 0.0" />
-			<parent link="femur_${side}${position}" />
-			<child link="tibia_${side}${position}" />
-			<axis xyz="0.0 0.0 ${axis}" />
-			<limit lower="${joint_lower_limit}" upper="${joint_upper_limit}" effort="${joint_effort}" velocity="${joint_velocity}" />
-		</joint>
-		<transmission name="tibia_transmission_${side}${position}">
-            <type>transmission_interface/SimpleTransmission</type>
-            <joint name="tibia_joint_${side}${position}">
-                <hardwareInterface>EffortJointInterface</hardwareInterface>
-            </joint>
-            <actuator name="tibia_motor_${side}${position}">
-                <hardwareInterface>EffortJointInterface</hardwareInterface>
-                <mechanicalReduction>1</mechanicalReduction>
-            </actuator>
+	<!-- tibia -->
+	<joint name="tibia_joint_${side}${position}" type="revolute">
+		<origin xyz="0.0 -${femur_length} 0.0" rpy="${pi} 0.0 0.0" />
+		<parent link="femur_${side}${position}" />
+		<child link="tibia_${side}${position}" />
+		<axis xyz="0.0 0.0 ${axis}" />
+		<limit lower="${joint_lower_limit}" upper="${joint_upper_limit}" effort="${joint_effort}" velocity="${joint_velocity}" />
+	</joint>
+	<transmission name="tibia_transmission_${side}${position}">
+        	<type>transmission_interface/SimpleTransmission</type>
+          	<joint name="tibia_joint_${side}${position}">
+                	<hardwareInterface>EffortJointInterface</hardwareInterface>
+            	</joint>
+            	<actuator name="tibia_motor_${side}${position}">
+                	<hardwareInterface>EffortJointInterface</hardwareInterface>
+                	<mechanicalReduction>1</mechanicalReduction>
+            	</actuator>
         </transmission>
         <link name="tibia_${side}${position}">
-            <visual>
-                <origin xyz="0.0 0.0 0.0" rpy="0.0 0.0 0.0"/>
-                <geometry>
-                    <mesh filename="package://phantom_description/meshes/phantomX/tibia.stl" scale="0.001 0.001 0.001"/>
-                </geometry>
-                <material name="">
-                    <color rgba="0.7 0.7 0.7 1"/>
-                </material>
-            </visual>
-            <collision>
-                <origin xyz="0.0 0.0 0.0" rpy="0.0 0.0 0.0" />
-                <geometry>
-                    <mesh filename="package://phantom_description/meshes/phantomX/tibia.stl" scale="0.001 0.001 0.001"/>
-                </geometry>
-                <material name="">
-                    <color rgba="0.7 0.7 0.7 1" />
-                </material>
-            </collision>
-            <inertial>
-                <origin xyz="0.0 0.0 0.0" rpy="0.0 0.0 0.0" />
-                <mass value="0.00001"/>
-                <inertia
-                    ixx="1.0" ixy="0.0"  ixz="0.0"
-                    iyy="1.0" iyz="0.0"
-                    izz="1.0" />
-            </inertial>
+        	<visual>
+                	<origin xyz="0.0 0.0 0.0" rpy="0.0 0.0 0.0"/>
+                	<geometry>
+                    		<mesh filename="package://phantom_description/meshes/phantomX/tibia.stl" scale="0.001 0.001 0.001"/>
+                	</geometry>
+                	<material name="">
+                   		<color rgba="0.7 0.7 0.7 1"/>
+                	</material>
+            	</visual>
+            	<collision>
+                	<origin xyz="0.0 0.0 0.0" rpy="0.0 0.0 0.0" />
+                	<geometry>
+                        	<mesh filename="package://phantom_description/meshes/phantomX/tibia.stl" scale="0.001 0.001 0.001"/>
+                	</geometry>
+                	<material name="">
+                    		<color rgba="0.7 0.7 0.7 1" />
+                	</material>
+            	</collision>
+            	<inertial>
+                	<origin xyz="0.0 0.0 0.0" rpy="0.0 0.0 0.0" />
+                	<mass value="0.00001"/>
+                	<inertia ixx="1.0" ixy="0.0"  ixz="0.0" iyy="1.0" iyz="0.0" izz="1.0" />
+            	</inertial>
         </link>
         <gazebo reference="tibia_${side}${position}">
-            <material>Gazebo/DarkGrey</material>
+        	<material>Gazebo/DarkGrey</material>
         </gazebo>
-	</xacro:macro>
+/xacro:macro>
 <!-- Build robot model -->
-	<xacro:leg side="R" position="R" x="-0.120" y="-0.060" angle="-${pi*3/4}" axis="1" />
-	<xacro:leg side="R" position="M" x="0.0" y="-0.100" angle="-${pi/2}" axis="1" />
-	<xacro:leg side="R" position="F" x="0.120" y="-0.060" angle="-${pi/4}" axis="1" />
-	<xacro:leg side="L" position="R" x="-0.120" y="0.060" angle="${pi*3/4}" axis="-1" />
-	<xacro:leg side="L" position="M" x="0.0" y="0.100" angle="${pi/2}" axis="-1" />
-	<xacro:leg side="L" position="F" x="0.120" y="0.060" angle="${pi/4}" axis="-1" />
+<xacro:leg side="R" position="R" x="-0.120" y="-0.060" angle="-${pi*3/4}" axis="1" />
+<xacro:leg side="R" position="M" x="0.0" y="-0.100" angle="-${pi/2}" axis="1" />
+<xacro:leg side="R" position="F" x="0.120" y="-0.060" angle="-${pi/4}" axis="1" />
+<xacro:leg side="L" position="R" x="-0.120" y="0.060" angle="${pi*3/4}" axis="-1" />
+<xacro:leg side="L" position="M" x="0.0" y="0.100" angle="${pi/2}" axis="-1" />
+<xacro:leg side="L" position="F" x="0.120" y="0.060" angle="${pi/4}" axis="-1" />
 </robot>
